Commit message: Rotate to add gravity to sac

File: experiments/robot_one_dof/models/one_dof.urdf (robot description, URDF)
Before this commit: robot one_dof, 4 links, 3 joints
Joints:
- joint joint_fixed: origin xyz=0.0 0.0 0.0 rpy=0.0 1.57 0.0 -> xyz=0.0 0.0 0.0 rpy=0.0 0 0.0

Commit message: Setup pybullet env with onedof

File: experiments/robot_one_dof/models/one_dof.urdf (robot description, URDF)
Before this commit: robot one_dof, 4 links, 3 joints
Joints:
- joint joint_1: limit lower=-3.14 upper=3.14 effort=10.0 velocity=1.0 -> lower=-3.14 upper=3.14 effort=20.0 velocity=3.14
- joint joint_fixed: origin xyz=0.0 0.0 0.0 rpy=0.0 0 0.0 -> xyz=0.0 0.0 0.0 rpy=0.0 -1.57 1.57
- joint joint_tcp: limit lower=-3.14 upper=3.14 effort=10.0 velocity=1.0 -> lower=-3.14 upper=3.14 effort=20.0 velocity=3.14
